Commit message: Added gripper

File: libot_description/urdf/arm.xacro (robot description, xacro)
@@ -27,4 +27,21 @@
     <xacro:cylinder_link name="horizontal_prismatic_link2" material="yellow" radius="0.03" length="0.16" />
     <xacro:cylinder_link name="horizontal_prismatic_link3" material="orange" radius="0.02" length="0.16" />
+    <link name="gripper_pitch_link">
+        <visual>
+            <geometry>
+                <cylinder radius="0.005" length="0.038" />
+            </geometry>
+            <origin xyz="0 0 0" rpy="${pi/2} 0 0" />
+            <material name="yellow" />
+        </visual>
+        <collision>
+            <geometry>
+                <cylinder radius="0.005" length="0.038"/>
+            </geometry>
+            <origin xyz="0 0 0" rpy="${pi/2} 0 0" />
+        </collision>
+    <xacro:cylinder_inertia m="0.3" r="0.005" h="0.038"
+                    o_xyz="0 0 0" o_rpy="${pi/2} 0 0" />
+    </link>
     <joint name="arm_base_prismatic1_joint" type="fixed">
         <parent link="arm_base_link" />
@@ -72,3 +89,11 @@
         <dynamics friction="0.3" damping="0.3" />
     </joint>
+    <joint name="horizontal_prismatic3_gripper_pitch_joint" type="revolute">
+        <parent link="horizontal_prismatic_link3" />
+        <child link="gripper_pitch_link" />
+        <origin xyz="0 0 0.16" rpy="0 0 0" />
+        <axis xyz="0 1 0" />
+        <limit lower="${-pi/2}" upper="${pi/2}" effort="100" velocity="100" />
+        <dynamics friction="0.3" damping="0.3" />
+    </joint>
 </robot>

File: libot_description/urdf/standalone_arm.urdf.xacro (robot description, xacro)
@@ -4,3 +4,12 @@
     <xacro:include filename="arm.xacro" />
     <xacro:include filename="arm_gazebo.xacro" />
+    <xacro:include filename="gripper.xacro" />
+    <joint name="gripper_pitch_base_joint" type="continuous">
+        <parent link="gripper_pitch_link" />
+        <child link="gripper_base_link" />
+        <origin xyz="0 0 0" rpy="0 0 ${pi/2}"/>
+        <axis xyz="0 0 1" />
+        <limit effort="100" velocity="100" />
+        <dynamics friction="0.3" damping="0.3" />
+    </joint>
 </robot>

Commit message: Adjusted some stuff for the gripper + now controllable in gazebo

File: libot_description/urdf/arm.xacro (robot description, xacro)
@@ -21,11 +21,12 @@
     </xacro:macro>
     <xacro:cylinder_link name="arm_base_link" material="yellow" radius="0.09" length="0.02" />
-    <xacro:cylinder_link name="vertical_prismatic_link1" material="orange" radius="0.07" length="0.2" />
-    <xacro:cylinder_link name="vertical_prismatic_link2" material="yellow" radius="0.06" length="0.2" />
-    <xacro:cylinder_link name="vertical_prismatic_link3" material="orange" radius="0.05" length="0.2" />
-    <xacro:cylinder_link name="horizontal_prismatic_link1" material="orange" radius="0.04" length="0.16" />
-    <xacro:cylinder_link name="horizontal_prismatic_link2" material="yellow" radius="0.03" length="0.16" />
-    <xacro:cylinder_link name="horizontal_prismatic_link3" material="orange" radius="0.02" length="0.16" />
-    <link name="gripper_pitch_link">
+    <xacro:cylinder_link name="vertical_prismatic_link1" material="orange" radius="0.07" length="0.35" />
+    <xacro:cylinder_link name="vertical_prismatic_link2" material="yellow" radius="0.06" length="0.35" />
+    <xacro:cylinder_link name="vertical_prismatic_link3" material="orange" radius="0.05" length="0.35" />
+    <xacro:cylinder_link name="horizontal_prismatic_link1" material="orange" radius="0.04" length="0.125" />
+    <xacro:cylinder_link name="horizontal_prismatic_link2" material="yellow" radius="0.03" length="0.125" />
+    <xacro:cylinder_link name="horizontal_prismatic_link3" material="orange" radius="0.02" length="0.125" />
+    <xacro:cylinder_link name="roll_link" material="greenish" radius="0.018" length="0.01" />
+    <link name="pitch_link">
         <visual>
             <geometry>
@@ -47,5 +48,5 @@
         <parent link="arm_base_link" />
         <child link="vertical_prismatic_link1" />
-        <origin xyz="0 0 0.02" rpy="0 0 0" />
+        <origin xyz="0 0 -0.1" rpy="0 0 0" />
         <axis xyz="0 0 1" />
     </joint>
@@ -55,5 +56,5 @@
         <origin xyz="0 0 0" rpy="0 0 0" />
         <axis xyz="0 0 1" />
-        <limit lower="0" upper="0.16" effort="100" velocity="100" />
+        <limit lower="0" upper="0.35" effort="100" velocity="100" />
         <dynamics friction="0.3" damping="0.3" />
     </joint>
@@ -64,5 +65,5 @@
         <axis xyz="0 0 1" />
         <mimic joint="vertical_prismatic1_2_joint" multiplier="1" offset="0"/>
-        <limit lower="0" upper="0.16" effort="100" velocity="100" />
+        <limit lower="0" upper="0.35" effort="100" velocity="100" />
         <dynamics friction="0.3" damping="0.3" />
     </joint>
@@ -70,5 +71,5 @@
         <parent link="vertical_prismatic_link3" />
         <child link="horizontal_prismatic_link1" />
-        <origin xyz="-0.03 0 ${0.2 - 0.05}" rpy="0 ${pi/2} 0" />
+        <origin xyz="-0.03 0 ${0.35 - 0.05}" rpy="0 ${pi/2} 0" />
     </joint>
     <joint name="horizontal_prismatic1_2_joint" type="prismatic">
@@ -77,5 +78,5 @@
         <origin xyz="0 0 0" rpy="0 0 0" />
         <axis xyz="0 0 1" />
-        <limit lower="0" upper="0.16" effort="100" velocity="100" />
+        <limit lower="0" upper="0.125" effort="100" velocity="100" />
         <dynamics friction="0.3" damping="0.3" />
     </joint>
@@ -86,11 +87,19 @@
         <axis xyz="0 0 1" />
         <mimic joint="horizontal_prismatic1_2_joint" multiplier="1" offset="0"/>
-        <limit lower="0" upper="0.16" effort="100" velocity="100" />
+        <limit lower="0" upper="0.1" effort="100" velocity="100" />
         <dynamics friction="0.3" damping="0.3" />
     </joint>
-    <joint name="horizontal_prismatic3_gripper_pitch_joint" type="revolute">
+    <joint name="horizontal_prismatic3_roll_joint" type="continuous">
         <parent link="horizontal_prismatic_link3" />
-        <child link="gripper_pitch_link" />
-        <origin xyz="0 0 0.16" rpy="0 0 0" />
+        <child link="roll_link" />
+        <origin xyz="0 0 0.125" rpy="0 0 0" />
+        <axis xyz="0 0 1" />
+        <limit effort="100" velocity="100" />
+        <dynamics friction="0.3" damping="0.3" />
+    </joint>
+    <joint name="roll_pitch_joint" type="revolute">
+        <parent link="roll_link" />
+        <child link="pitch_link" />
+        <origin xyz="0 0 0.01" rpy="0 0 0" />
         <axis xyz="0 1 0" />
         <limit lower="${-pi/2}" upper="${pi/2}" effort="100" velocity="100" />

File: libot_description/urdf/arm_gazebo.xacro (robot description, xacro)
@@ -9,11 +9,6 @@
             <joint_name>horizontal_prismatic1_2_joint</joint_name>
             <joint_name>horizontal_prismatic2_3_joint</joint_name>
-        </plugin>
-    </gazebo>
-    <gazebo>
-        <plugin
-            filename="gz-sim-joint-controller-system"
-            name="gz::sim::systems::JointController">
-            <joint_name>base_left_wheel_joint</joint_name>
+            <joint_name>horizontal_prismatic3_roll_joint</joint_name>
+            <joint_name>roll_pitch_joint</joint_name>
         </plugin>
     </gazebo>
@@ -32,3 +27,17 @@
         </plugin>
     </gazebo>
+    <gazebo>
+        <plugin
+            filename="gz-sim-joint-controller-system"
+            name="gz::sim::systems::JointController">
+            <joint_name>horizontal_prismatic3_roll_joint</joint_name>
+        </plugin>
+    </gazebo>
+    <gazebo>
+        <plugin
+            filename="gz-sim-joint-controller-system"
+            name="gz::sim::systems::JointController">
+            <joint_name>roll_pitch_joint</joint_name>
+        </plugin>
+    </gazebo>
 </robot>

File: libot_description/urdf/camera.xacro (robot description, xacro)
@@ -25,5 +25,5 @@
         <parent link="base_link" />
         <child link="camera_link" />
-        <origin xyz="${base_length / 2.0 + 0.05} 0 ${base_height / 2.0}" rpy="0 0 0"/>
+        <origin xyz="${base_length / 2.0 + 0.005} 0 ${base_height / 2.0}" rpy="0 0 0"/>
     </joint>
     <!-- generate an optical frame

File: libot_description/urdf/common_properties.xacro (robot description, xacro)
@@ -12,4 +12,7 @@
     <material name="yellow">
         <color rgba="1.0 0.65 0.1  1" /> <!-- r g b alpha -->
+    </material>
+    <material name="greenish">
+        <color rgba="0.9 0.75 0.1  1" /> <!-- r g b alpha -->
     </material>
     <xacro:macro name="box_inertia" params="m x y z o_xyz o_rpy">

File: libot_description/urdf/gripper.xacro (robot description, xacro)
@@ -15,9 +15,6 @@
             <origin xyz="0 0 0.01" rpy="0 0 0"/>
         </collision>
-        <!-- <inertial>
-            <mass value="0.1"/>
-            <origin xyz="0 0 0" rpy="0 0 0"/>
-            <inertia ixx="0.0001" ixy="0.0" ixz="0.0" iyy="0.0001" iyz="0.0" izz="0.0001"/>
-        </inertial> -->
+        <xacro:box_inertia m="0.1" x="0.2" y="0.06" z="0.02"
+                        o_xyz="0 0 0.01" o_rpy="0 0 0" />
     </link>
     <link name="gripper_left_finger_link">
@@ -35,9 +32,6 @@
             <origin xyz="0 0 0.04" rpy="0 0 0"/>
         </collision>
-        <!-- <inertial>
-            <mass value="0.05"/>
-            <origin xyz="0 0 0" rpy="0 0 0"/>
-            <inertia ixx="0.00005" ixy="0.0" ixz="0.0" iyy="0.00005" iyz="0.0" izz="0.00005"/>
-        </inertial> -->
+        <xacro:box_inertia m="0.1" x="0.02" y="0.06" z="0.08"
+                        o_xyz="0 0 0.04" o_rpy="0 0 0" />
     </link>
     <joint name="gripper_left_finger_joint" type="prismatic">
@@ -47,5 +41,5 @@
         <axis xyz="1 0 0"/>
         <limit lower="0" upper="0.06" effort="1000.0" velocity="1.0"/>
-        <!-- <dynamics damping="0.1" friction="0.1"/> -->
+        <dynamics damping="0.1" friction="0.1"/>
     </joint>
     <link name="gripper_right_finger_link">
@@ -63,9 +57,6 @@
             <origin xyz="0 0 0.04" rpy="0 0 0"/>
         </collision>
-        <!-- <inertial>
-            <mass value="0.05"/>
-            <origin xyz="0 0 0" rpy="0 0 0"/>
-            <inertia ixx="0.00005" ixy="0.0" ixz="0.0" iyy="0.00005" iyz="0.0" izz="0.00005"/>
-        </inertial> -->
+        <xacro:box_inertia m="0.1" x="0.02" y="0.06" z="0.08"
+                        o_xyz="0 0 0.04" o_rpy="0 0 0" />
     </link>
     <joint name="gripper_right_finger_joint" type="prismatic">
@@ -76,5 +67,5 @@
         <mimic joint="gripper_left_finger_joint" multiplier="1" offset="0"/>
         <limit lower="0.0" upper="0.06" effort="1000.0" velocity="1.0"/>
-        <!-- <dynamics damping="0.1" friction="0.1"/> -->
+        <dynamics damping="0.1" friction="0.1"/>
     </joint>
 </robot>

File: libot_description/urdf/libot.urdf.xacro (robot description, xacro)
@@ -10,5 +10,5 @@
         <parent link="base_link" />
         <child link="arm_base_link" />
-        <origin xyz="${base_length / 4.0} 0 ${base_height}" rpy="0 0 0"/>
+        <origin xyz="${base_length / 3.5} 0 ${base_height}" rpy="0 0 0"/>
         <axis xyz="0 0 1" />
         <limit effort="100" velocity="100" />

File: libot_description/urdf/libot_base.xacro (robot description, xacro)
@@ -2,8 +2,8 @@
 <robot xmlns:xacro="http://www.ros.org/wiki/xacro">
     <!-- Body Variables -->
-    <xacro:property name="base_length" value="0.7" />
-    <xacro:property name="base_width" value="0.4" />
-    <xacro:property name="base_height" value="0.215" />
-    <xacro:property name="wheel_radius" value="0.1" />
+    <xacro:property name="base_length" value="0.65" />
+    <xacro:property name="base_width" value="0.425" />
+    <xacro:property name="base_height" value="0.205" />
+    <xacro:property name="wheel_radius" value="0.05" />
     <xacro:property name="wheel_length" value="0.05" />
     <xacro:property name="caster_radius" value="${wheel_radius / 2.0}" />
@@ -59,5 +59,5 @@
         <parent link="base_link" />
         <child link="back_right_wheel_link" />
-        <origin xyz="${-base_length / 3.5} ${-(base_width + wheel_length) / 2.0} 0" rpy="-${pi / 2.0} 0 0"/>
+        <origin xyz="${-base_length / 3.0} ${-(base_width - wheel_length - 0.02) / 2.0} 0" rpy="-${pi / 2.0} 0 0"/>
         <axis xyz="0 0 1" />
     </joint>
@@ -65,5 +65,5 @@
         <parent link="base_link" />
         <child link="back_left_wheel_link" />
-        <origin xyz="${-base_length / 3.5} ${(base_width + wheel_length) / 2.0} 0" rpy="-${pi / 2.0} 0 0"/>
+        <origin xyz="${-base_length / 3.0} ${(base_width - wheel_length - 0.02) / 2.0} 0" rpy="-${pi / 2.0} 0 0"/>
         <axis xyz="0 0 1" />
     </joint>
@@ -71,5 +71,5 @@
         <parent link="base_link" />
         <child link="front_right_wheel_link" />
-        <origin xyz="${base_length / 3.5} ${-(base_width + wheel_length) / 2.0} 0" rpy="-${pi / 2.0} 0 0"/>
+        <origin xyz="${base_length / 3.0} ${-(base_width - wheel_length - 0.02) / 2.0} 0" rpy="-${pi / 2.0} 0 0"/>
         <axis xyz="0 0 1" />
     </joint>
@@ -77,5 +77,5 @@
         <parent link="base_link" />
         <child link="front_left_wheel_link" />
-        <origin xyz="${base_length / 3.5} ${(base_width + wheel_length) / 2.0} 0" rpy="-${pi / 2.0} 0 0"/>
+        <origin xyz="${base_length / 3.0} ${(base_width - wheel_length - 0.02) / 2.0} 0" rpy="-${pi / 2.0} 0 0"/>
         <axis xyz="0 0 1" />
     </joint>

File: libot_description/urdf/standalone_arm.urdf.xacro (robot description, xacro)
@@ -5,6 +5,7 @@
     <xacro:include filename="arm_gazebo.xacro" />
     <xacro:include filename="gripper.xacro" />
-    <joint name="gripper_pitch_base_joint" type="continuous">
-        <parent link="gripper_pitch_link" />
+    <xacro:include filename="gripper_gazebo.xacro" />
+    <joint name="pitch_gripper_joint" type="fixed">
+        <parent link="pitch_link" />
         <child link="gripper_base_link" />
         <origin xyz="0 0 0" rpy="0 0 ${pi/2}"/>
